Commit message: fixed broken config

File: mrv1a_description/config/mrv1a.config.xacro (robot description, xacro)
@@ -1,5 +1,11 @@
 <?xml version="1.0"?>
 <robot xmlns:xacro="http://www.ros.org/wiki/xacro" name="mrv1a">
-    <xacro:arg name="initial_positions_file" default="$(find mrv1a_description)/config/initial_positions.yaml" />
+    <!-- Enable setting arguments from the launch file -->
+    <xacro:arg name="use_sim" default="false" />
+    <xacro:arg name="use_fake_hardware" default="true" />
+    <xacro:arg name="prefix" default="" />
+    <xacro:arg name="robot_ip" default="192.168.122.200" />
+    <xacro:arg name="robot_port" default="10000" />
+    <xacro:arg name="initial_positions_file" default="initial_positions.yaml" />
     <!-- Import mrv1a urdf file -->
     <xacro:include filename="$(find mrv1a_description)/urdf/mrv1a.urdf.xacro" />

File: mrv1a_description/ros2_control/mrv1a.r2c_hardware.xacro (robot description, xacro)
@@ -1,8 +1,8 @@
 <?xml version="1.0"?>
 <robot xmlns:xacro="http://www.ros.org/wiki/xacro">
-    <xacro:macro name="iiwa_r2c_hardware" params="name prefix robot_ip robot_port initial_positions_file use_sim:=^|false use_fake_hardware:=^|true">
+    <xacro:macro name="mrv1a_r2c_hardware" params="name prefix robot_ip robot_port initial_positions_file use_sim:=^|false use_fake_hardware:=^|true">
         <xacro:property name="initial_positions" value="${load_yaml(initial_positions_file)['initial_positions']}"/>
         <ros2_control name="${name}" type="system">
-            <<xacro:if value="$(arg use_sim)">
+            <xacro:if value="$(arg use_sim)">
                 <hardware>
                     <plugin>gazebo_ros2_control/GazeboSystem</plugin>

File: mrv1a_description/urdf/mrv1a.urdf.xacro (robot description, xacro)
@@ -5,5 +5,143 @@
       <color rgba="0.5 0.5 0.5 1.0"/>
     </material>
-    <link name="${prefix}mrv1a_base" type="fixed"/>
+    <link name="${prefix}mrv1a_base">
+        <visual>
+          <origin rpy="0 0 0" xyz="0 0 0"/>
+          <geometry>
+            <mesh filename="package://mrv1a_description/meshes/body1_0.stl" scale="0.001 0.001 0.001"/>
+          </geometry>
+          <material name="gray"/>
+        </visual>
+        <collision>
+          <origin rpy="0 0 0" xyz="0 0 0"/>
+          <geometry>
+            <mesh filename="package://mrv1a_description/meshes/body1_0.stl" scale="0.001 0.001 0.001"/>
+          </geometry>
+        </collision>
+        <inertial>
+            <mass value="1"/>
+            <inertia ixx="1.0" ixy="0.0" ixz="0.0" iyy="1.0" iyz="0.0" izz="1.0"/>
+        </inertial>
+    </link>
+    <link name="${prefix}link_1">
+        <visual>
+          <origin rpy="0 0 0" xyz="0 0 0"/>
+          <geometry>
+            <mesh filename="package://mrv1a_description/meshes/body1_1.stl" scale="0.001 0.001 0.001"/>
+          </geometry>
+          <material name="gray"/>
+        </visual>
+        <collision>
+          <origin rpy="0 0 0" xyz="0 0 0"/>
+          <geometry>
+            <mesh filename="package://mrv1a_description/meshes/body1_1.stl" scale="0.001 0.001 0.001"/>
+          </geometry>
+        </collision>
+        <inertial>
+          <mass value="1"/>
+          <inertia ixx="1.0" ixy="0.0" ixz="0.0" iyy="1.0" iyz="0.0" izz="1.0"/>
+        </inertial>
+    </link>
+    <link name="${prefix}link_2">
+        <visual>
+          <origin rpy="0 0 -1.57" xyz="0 -0.25 0"/>
+          <geometry>
+            <mesh filename="package://mrv1a_description/meshes/body1_2.stl" scale="0.001 0.001 0.001"/>
+          </geometry>
+          <material name="gray"/>
+        </visual>
+        <collision>
+          <origin rpy="0 0 -1.57" xyz="0 -0.25 0"/>
+          <geometry>
+            <mesh filename="package://mrv1a_description/meshes/body1_2.stl" scale="0.001 0.001 0.001"/>
+          </geometry>
+        </collision>
+        <inertial>
+          <mass value="1"/>
+          <inertia ixx="1.0" ixy="0.0" ixz="0.0" iyy="1.0" iyz="0.0" izz="1.0"/>
+        </inertial>
+    </link>
+    <link name="${prefix}link_3">
+        <visual>
+          <origin rpy="1.57 0 0" xyz="-0.09 0 0"/>
+          <geometry>
+            <mesh filename="package://mrv1a_description/meshes/body1_3.stl" scale="0.001 0.001 0.001"/>
+          </geometry>
+          <material name="gray"/>
+        </visual>
+        <collision>
+          <origin rpy="1.57 0 0" xyz="-0.09 0 0"/>
+          <geometry>
+            <mesh filename="package://mrv1a_description/meshes/body1_3.stl" scale="0.001 0.001 0.001"/>
+          </geometry>
+        </collision>
+        <inertial>
+          <mass value="1"/>
+          <inertia ixx="1.0" ixy="0.0" ixz="0.0" iyy="1.0" iyz="0.0" izz="1.0"/>
+        </inertial>
+    </link>
+    <link name="${prefix}link_4">
+        <visual>
+          <origin rpy="-1.57 0 0" xyz="0 0 0"/>
+          <geometry>
+            <mesh filename="package://mrv1a_description/meshes/body1_4.stl" scale="0.001 0.001 0.001"/>
+          </geometry>
+          <material name="gray"/>
+        </visual>
+        <collision>
+          <origin rpy="0 0 0" xyz="0 0 0"/>
+          <geometry>
+            <mesh filename="package://mrv1a_description/meshes/body1_4.stl" scale="0.001 0.001 0.001"/>
+          </geometry>
+        </collision>
+        <inertial>
+          <mass value="1"/>
+          <inertia ixx="1.0" ixy="0.0" ixz="0.0" iyy="1.0" iyz="0.0" izz="1.0"/>
+        </inertial>
+    </link>
+    <link name="${prefix}link_5">
+        <visual>
+          <origin rpy="1.57 0 0" xyz="0 0 0"/>
+          <geometry>
+            <mesh filename="package://mrv1a_description/meshes/body1_5.stl" scale="0.001 0.001 0.001"/>
+          </geometry>
+          <material name="gray"/>
+        </visual>
+        <collision>
+          <origin rpy="0 0 0" xyz="0 0 0"/>
+          <geometry>
+            <mesh filename="package://mrv1a_description/meshes/body1_5.stl" scale="0.001 0.001 0.001"/>
+          </geometry>
+        </collision>
+        <inertial>
+          <mass value="1"/>
+          <inertia ixx="1.0" ixy="0.0" ixz="0.0" iyy="1.0" iyz="0.0" izz="1.0"/>
+        </inertial>
+    </link>
+    <link name="${prefix}link_6">
+        <visual>
+          <origin rpy="0 0 0" xyz="0 0 0"/>
+          <geometry>
+            <mesh filename="package://mrv1a_description/meshes/body1_6.stl" scale="0.001 0.001 0.001"/>
+          </geometry>
+          <material name="gray"/>
+        </visual>
+        <collision>
+          <origin rpy="0 0 0" xyz="0 0 0"/>
+          <geometry>
+            <mesh filename="package://mrv1a_description/meshes/body1_6.stl" scale="0.001 0.001 0.001"/>
+          </geometry>
+        </collision>
+        <inertial>
+          <mass value="1"/>
+          <inertia ixx="1.0" ixy="0.0" ixz="0.0" iyy="1.0" iyz="0.0" izz="1.0"/>
+        </inertial>
+    </link>
+    <link name="${prefix}tool0">
+      <inertial>
+          <mass value="1"/>
+          <inertia ixx="1.0" ixy="0.0" ixz="0.0" iyy="1.0" iyz="0.0" izz="1.0"/>
+        </inertial>
+    </link>
     <joint name="${prefix}mrv1a_base" type="fixed">
         <xacro:insert_block name="origin" />
@@ -11,143 +149,4 @@
         <child link="${prefix}mrv1a_base"/>
     </joint>
-    <link name="${prefix}mrv1a_base">
-        <visual>
-          <origin rpy="0 0 0" xyz="0 0 0"/>
-          <geometry>
-            <mesh filename="package://mrv1a_description/meshes/body1_0.stl" scale="0.001 0.001 0.001"/>
-          </geometry>
-          <material name="gray"/>
-        </visual>
-        <collision>
-          <origin rpy="0 0 0" xyz="0 0 0"/>
-          <geometry>
-            <mesh filename="package://mrv1a_description/meshes/body1_0.stl" scale="0.001 0.001 0.001"/>
-          </geometry>
-        </collision>
-        <inertial>
-            <mass value="1"/>
-            <inertia ixx="1.0" ixy="0.0" ixz="0.0" iyy="1.0" iyz="0.0" izz="1.0"/>
-        </inertial>
-    </link>
-    <link name="${prefix}link_1">
-        <visual>
-          <origin rpy="0 0 0" xyz="0 0 0"/>
-          <geometry>
-            <mesh filename="package://mrv1a_description/meshes/body1_1.stl" scale="0.001 0.001 0.001"/>
-          </geometry>
-          <material name="gray"/>
-        </visual>
-        <collision>
-          <origin rpy="0 0 0" xyz="0 0 0"/>
-          <geometry>
-            <mesh filename="package://mrv1a_description/meshes/body1_1.stl" scale="0.001 0.001 0.001"/>
-          </geometry>
-        </collision>
-        <inertial>
-          <mass value="1"/>
-          <inertia ixx="1.0" ixy="0.0" ixz="0.0" iyy="1.0" iyz="0.0" izz="1.0"/>
-        </inertial>
-    </link>
-    <link name="${prefix}link_2">
-        <visual>
-          <origin rpy="0 0 -1.57" xyz="0 -0.25 0"/>
-          <geometry>
-            <mesh filename="package://mrv1a_description/meshes/body1_2.stl" scale="0.001 0.001 0.001"/>
-          </geometry>
-          <material name="gray"/>
-        </visual>
-        <collision>
-          <origin rpy="0 0 -1.57" xyz="0 -0.25 0"/>
-          <geometry>
-            <mesh filename="package://mrv1a_description/meshes/body1_2.stl" scale="0.001 0.001 0.001"/>
-          </geometry>
-        </collision>
-        <inertial>
-          <mass value="1"/>
-          <inertia ixx="1.0" ixy="0.0" ixz="0.0" iyy="1.0" iyz="0.0" izz="1.0"/>
-        </inertial>
-    </link>
-    <link name="${prefix}link_3">
-        <visual>
-          <origin rpy="1.57 0 0" xyz="-0.09 0 0"/>
-          <geometry>
-            <mesh filename="package://mrv1a_description/meshes/body1_3.stl" scale="0.001 0.001 0.001"/>
-          </geometry>
-          <material name="gray"/>
-        </visual>
-        <collision>
-          <origin rpy="1.57 0 0" xyz="-0.09 0 0"/>
-          <geometry>
-            <mesh filename="package://mrv1a_description/meshes/body1_3.stl" scale="0.001 0.001 0.001"/>
-          </geometry>
-        </collision>
-        <inertial>
-          <mass value="1"/>
-          <inertia ixx="1.0" ixy="0.0" ixz="0.0" iyy="1.0" iyz="0.0" izz="1.0"/>
-        </inertial>
-    </link>
-    <link name="${prefix}link_4">
-        <visual>
-          <origin rpy="-1.57 0 0" xyz="0 0 0"/>
-          <geometry>
-            <mesh filename="package://mrv1a_description/meshes/body1_4.stl" scale="0.001 0.001 0.001"/>
-          </geometry>
-          <material name="gray"/>
-        </visual>
-        <collision>
-          <origin rpy="0 0 0" xyz="0 0 0"/>
-          <geometry>
-            <mesh filename="package://mrv1a_description/meshes/body1_4.stl" scale="0.001 0.001 0.001"/>
-          </geometry>
-        </collision>
-        <inertial>
-          <mass value="1"/>
-          <inertia ixx="1.0" ixy="0.0" ixz="0.0" iyy="1.0" iyz="0.0" izz="1.0"/>
-        </inertial>
-    </link>
-    <link name="${prefix}link_5">
-        <visual>
-          <origin rpy="1.57 0 0" xyz="0 0 0"/>
-          <geometry>
-            <mesh filename="package://mrv1a_description/meshes/body1_5.stl" scale="0.001 0.001 0.001"/>
-          </geometry>
-          <material name="gray"/>
-        </visual>
-        <collision>
-          <origin rpy="0 0 0" xyz="0 0 0"/>
-          <geometry>
-            <mesh filename="package://mrv1a_description/meshes/body1_5.stl" scale="0.001 0.001 0.001"/>
-          </geometry>
-        </collision>
-        <inertial>
-          <mass value="1"/>
-          <inertia ixx="1.0" ixy="0.0" ixz="0.0" iyy="1.0" iyz="0.0" izz="1.0"/>
-        </inertial>
-    </link>
-    <link name="${prefix}link_6">
-        <visual>
-          <origin rpy="0 0 0" xyz="0 0 0"/>
-          <geometry>
-            <mesh filename="package://mrv1a_description/meshes/body1_6.stl" scale="0.001 0.001 0.001"/>
-          </geometry>
-          <material name="gray"/>
-        </visual>
-        <collision>
-          <origin rpy="0 0 0" xyz="0 0 0"/>
-          <geometry>
-            <mesh filename="package://mrv1a_description/meshes/body1_6.stl" scale="0.001 0.001 0.001"/>
-          </geometry>
-        </collision>
-        <inertial>
-          <mass value="1"/>
-          <inertia ixx="1.0" ixy="0.0" ixz="0.0" iyy="1.0" iyz="0.0" izz="1.0"/>
-        </inertial>
-    </link>
-    <link name="${prefix}tool0">
-      <inertial>
-          <mass value="1"/>
-          <inertia ixx="1.0" ixy="0.0" ixz="0.0" iyy="1.0" iyz="0.0" izz="1.0"/>
-        </inertial>
-    </link>
     <joint name="${prefix}joint_a1" type="revolute">
         <origin rpy="-1.57 0 0" xyz="0 0 0.3"/>
